Commit message: velodyne乗っけた

File: turtlebot3_description/urdf/turtlebot3_burger.urdf.xacro (robot description, xacro)
@@ -140,3 +140,7 @@
     </inertial>
   </link>
+  <xacro:include filename="$(find velodyne_description)/urdf/HDL-32E.urdf.xacro"/>
+  <xacro:HDL-32E parent="base_link" name="velodyne" topic="/velodyne_points" hz="10" samples="220">
+    <origin xyz="-0.05 0 1.0" rpy="0 0 0" />
+  </xacro:HDL-32E>
 </robot>
