Commit message: made urdffile for burger

File: turtlebot3_description/urdf/turtlebot3_burger.gazebo.xacro (robot description, xacro)
@@ -108,5 +108,6 @@
         </scan>
         <range>
-          <min>0.120</min>
+          <min>0.105</min>
+          <!-- <min>0.120</min> -->
           <max>3.5</max>
           <resolution>0.015</resolution>

File: turtlebot3_description/urdf/turtlebot3_burger.urdf.xacro (robot description, xacro)
@@ -17,5 +17,5 @@
       <material name="light_black"/>
     </visual>
-    <collision>
+    <collision name="turtlebot3_contact">
       <origin xyz="-0.032 0 0.070" rpy="0 0 0"/>
       <geometry>
